File: esp-12ef-ver1/esp12ef-ver1.sch (KiCad schematic (older format))
At the start: 18 parts, among them J1 Battery, J2 USB-TTL, J3 BME280_CONNECTOR, SW1 RESET, U1 ESP-12F

Commit message: pcb done
Parts:
- C1, C2: footprint (none) -> Capacitor_THT:CP_Radial_D4.0mm_P2.00mm
- C3: footprint (none) -> Capacitor_THT:C_Disc_D4.3mm_W1.9mm_P5.00mm
- J1: footprint (none) -> Connector_PinHeader_2.54mm:PinHeader_1x02_P2.54mm_Vertical
- L1: footprint (none) -> Package_TO_SOT_THT:TO-92
- R1, R2, R3, R4, R5, R6, R7, R8, R9: footprint (none) -> Resistor_THT:R_Axial_DIN0207_L6.3mm_D2.5mm_P10.16mm_Horizontal
- SW1: footprint (none) -> Button_Switch_THT:SW_PUSH_6mm
- U1: footprint (none) -> ESP8266:ESP-12E
Changed lines of the file:
@@
 F 0 "U1" H 5650 4500 50  0000 C CNN
 F 1 "ESP-12F" H 5650 4400 50  0000 C CNN
-F 2 "" H 5650 3650 50  0001 C CNN
+F 2 "ESP8266:ESP-12E" H 5650 3650 50  0001 C CNN
 F 3 "" H 5650 3650 50  0001 C CNN
 	1    5650 3650
@@
 F 0 "R5" H 4620 2746 50  0000 L CNN
 F 1 "10k" H 4620 2655 50  0000 L CNN
-F 2 "" V 4480 2700 50  0001 C CNN
+F 2 "Resistor_THT:R_Axial_DIN0207_L6.3mm_D2.5mm_P10.16mm_Horizontal" V 4480 2700 50  0001 C CNN
 F 3 "~" H 4550 2700 50  0001 C CNN
 	1    4550 2700
@@
 F 0 "R6" H 6970 2746 50  0000 L CNN
 F 1 "10k" H 6970 2655 50  0000 L CNN
-F 2 "" V 6830 2700 50  0001 C CNN
+F 2 "Resistor_THT:R_Axial_DIN0207_L6.3mm_D2.5mm_P10.16mm_Horizontal" V 6830 2700 50  0001 C CNN
 F 3 "~" H 6900 2700 50  0001 C CNN
 	1    6900 2700
@@
 F 0 "R3" H 4120 2746 50  0000 L CNN
 F 1 "10k" H 4120 2655 50  0000 L CNN
-F 2 "" V 3980 2700 50  0001 C CNN
+F 2 "Resistor_THT:R_Axial_DIN0207_L6.3mm_D2.5mm_P10.16mm_Horizontal" V 3980 2700 50  0001 C CNN
 F 3 "~" H 4050 2700 50  0001 C CNN
 	1    4050 2700
@@
 F 0 "R9" H 7470 2746 50  0000 L CNN
 F 1 "10k" H 7470 2655 50  0000 L CNN
-F 2 "" V 7330 2700 50  0001 C CNN
+F 2 "Resistor_THT:R_Axial_DIN0207_L6.3mm_D2.5mm_P10.16mm_Horizontal" V 7330 2700 50  0001 C CNN
 F 3 "~" H 7400 2700 50  0001 C CNN
 	1    7400 2700
@@
 F 0 "R7" H 6970 4396 50  0000 L CNN
 F 1 "10k" H 6970 4305 50  0000 L CNN
-F 2 "" V 6830 4350 50  0001 C CNN
+F 2 "Resistor_THT:R_Axial_DIN0207_L6.3mm_D2.5mm_P10.16mm_Horizontal" V 6830 4350 50  0001 C CNN
 F 3 "~" H 6900 4350 50  0001 C CNN
 	1    6900 4350
@@
 F 0 "C3" H 4865 4446 50  0000 L CNN
 F 1 "0.1mF" H 4865 4355 50  0000 L CNN
-F 2 "" H 4788 4250 50  0001 C CNN
+F 2 "Capacitor_THT:C_Disc_D4.3mm_W1.9mm_P5.00mm" H 4788 4250 50  0001 C CNN
 F 3 "~" H 4750 4400 50  0001 C CNN
 	1    4750 4400
@@
 F 0 "SW1" H 4050 4585 50  0000 C CNN
 F 1 "RESET" H 4050 4494 50  0000 C CNN
-F 2 "" H 4050 4500 50  0001 C CNN
+F 2 "Button_Switch_THT:SW_PUSH_6mm" H 4050 4500 50  0001 C CNN
 F 3 "" H 4050 4500 50  0001 C CNN
 	1    4050 4300
@@
 F 0 "R8" V 6943 3750 50  0000 C CNN
 F 1 "470" V 7034 3750 50  0000 C CNN
-F 2 "" V 7080 3750 50  0001 C CNN
+F 2 "Resistor_THT:R_Axial_DIN0207_L6.3mm_D2.5mm_P10.16mm_Horizontal" V 7080 3750 50  0001 C CNN
 F 3 "~" H 7150 3750 50  0001 C CNN
 	1    7150 3750
@@
 F 0 "R4" V 4400 3550 50  0000 C CNN
 F 1 "470" V 4400 3700 50  0000 C CNN
-F 2 "" V 4230 3650 50  0001 C CNN
+F 2 "Resistor_THT:R_Axial_DIN0207_L6.3mm_D2.5mm_P10.16mm_Horizontal" V 4230 3650 50  0001 C CNN
 F 3 "~" H 4300 3650 50  0001 C CNN
 	1    4300 3650
@@
 F 0 "L1" H 3150 2947 60  0000 C CNN
 F 1 "HT7333-A" H 3150 2841 60  0000 C CNN
-F 2 "" H 3100 2550 60  0001 C CNN
+F 2 "Package_TO_SOT_THT:TO-92" H 3100 2550 60  0001 C CNN
 F 3 "" H 3100 2550 60  0000 C CNN
 	1    3100 2550
@@
 F 0 "C2" H 4468 4446 50  0000 L CNN
 F 1 "10mF" H 4468 4355 50  0000 L CNN
-F 2 "" H 4388 4250 50  0001 C CNN
+F 2 "Capacitor_THT:CP_Radial_D4.0mm_P2.00mm" H 4388 4250 50  0001 C CNN
 F 3 "~" H 4350 4400 50  0001 C CNN
 	1    4350 4400
@@
 F 0 "C1" H 2818 4446 50  0000 L CNN
 F 1 "10mF" H 2818 4355 50  0000 L CNN
-F 2 "" H 2738 4250 50  0001 C CNN
+F 2 "Capacitor_THT:CP_Radial_D4.0mm_P2.00mm" H 2738 4250 50  0001 C CNN
 F 3 "~" H 2700 4400 50  0001 C CNN
 	1    2700 4400
@@
 F 0 "J1" H 2006 2575 50  0000 C CNN
 F 1 "Battery" H 2006 2484 50  0000 C CNN
-F 2 "" H 2150 2450 50  0001 C CNN
+F 2 "Connector_PinHeader_2.54mm:PinHeader_1x02_P2.54mm_Vertical" H 2150 2450 50  0001 C CNN
 F 3 "" H 2150 2450 50  0001 C CNN
 	1    2150 2450
@@
 F 0 "R1" H 2420 3046 50  0000 L CNN
 F 1 "200k" H 2420 2955 50  0000 L CNN
-F 2 "" V 2280 3000 50  0001 C CNN
+F 2 "Resistor_THT:R_Axial_DIN0207_L6.3mm_D2.5mm_P10.16mm_Horizontal" V 2280 3000 50  0001 C CNN
 F 3 "~" H 2350 3000 50  0001 C CNN
 	1    2350 3000
@@
 F 0 "R2" H 2420 3946 50  0000 L CNN
 F 1 "800k" H 2420 3855 50  0000 L CNN
-F 2 "" V 2280 3900 50  0001 C CNN
+F 2 "Resistor_THT:R_Axial_DIN0207_L6.3mm_D2.5mm_P10.16mm_Horizontal" V 2280 3900 50  0001 C CNN
 F 3 "~" H 2350 3900 50  0001 C CNN
 	1    2350 3900

Commit message: уменьшен размер платы
Parts:
- L1: footprint Package_TO_SOT_THT:TO-92 -> ht7333-a:ht7333-a
Changed lines of the file:
@@
 F 0 "L1" H 3150 2947 60  0000 C CNN
 F 1 "HT7333-A" H 3150 2841 60  0000 C CNN
-F 2 "Package_TO_SOT_THT:TO-92" H 3100 2550 60  0001 C CNN
+F 2 "ht7333-a:ht7333-a" H 3100 2550 60  0001 C CNN
 F 3 "" H 3100 2550 60  0000 C CNN
 	1    3100 2550
