File: esp-12ef-smd/esp-12ef-smd.kicad_pcb (KiCad board)
At the start: 2 copper layers, 18 parts, among them J1 Battery, J2 USB-TTL, J3 BME280_CONNECTOR, SW1 RESET, U1 ESP-12F

Commit message: minor changes
Parts:
- added J4: 6PIN-WITH-POWER, Connector_PinSocket_2.54mm:PinSocket_1x06_P2.54mm_Vertical, B.Cu at (87.6, 92.7)
- J3: value BME280_CONNECTOR -> 6PIN-WITH-POWER; footprint Connector_PinSocket_2.54mm:PinSocket_1x04_P2.54mm_Vertical -> Connector_PinSocket_2.54mm:PinSocket_1x06_P2.54mm_Vertical; moved to B.Cu
- L1, SW1: moved to B.Cu
- moved J3 107.2 mm to (68.6, 67.3), turned to 180 degrees
- moved R9 69.9 mm to (108.0, 83.8)
- moved C3 62.1 mm to (69.8, 50.8), turned to 90 degrees
- moved C1 59.6 mm to (85.1, 50.8), turned to 90 degrees
- moved J2 58.8 mm to (115.6, 61.0)
- moved R3 58.2 mm to (80.3, 73.7), turned to 0 degrees
- moved R7 55.2 mm to (109.2, 74.9), turned to 0 degrees
- moved U1 53.4 mm to (87.4, 65.9)
- moved R5 51.1 mm to (80.0, 69.8), turned to 0 degrees
- moved C2 50.6 mm to (74.9, 50.8), turned to 90 degrees
- moved R8 50.4 mm to (108.0, 80.0), turned to 0 degrees
- moved R6 49.8 mm to (97.8, 87.6), turned to 0 degrees
- moved R4 49.4 mm to (80.0, 82.5), turned to 0 degrees
- moved R2 48.3 mm to (80.0, 64.8)
- moved J1 45.1 mm to (68.6, 58.4)
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Connections:
- J3 pad 2: Net-(C1-Pad2) -> GPIO14
- J3 pad 3: SCL -> GPIO13
- J3 pad 4: SDA -> GPIO12
- U1 pad 13: SDA -> GPIO4
- U1 pad 14: SCL -> GPIO5
- U1 pad 19: Net-(U1-Pad19) -> GPIO9
- U1 pad 20: Net-(U1-Pad20) -> GPIO10
- U1 pad 5: Net-(U1-Pad5) -> GPIO14
- U1 pad 6: Net-(U1-Pad6) -> GPIO12
- U1 pad 7: Net-(U1-Pad7) -> GPIO13
Routing:
- net Net-(C2-Pad1): track 87.2 -> 0.00 mm
- net Net-(C1-Pad1): track 61.0 -> 0.00 mm
- net Net-(C1-Pad2): track 144.7 -> 193.4 mm
- net Net-(J2-Pad2): track 46.9 -> 0.00 mm
- net Net-(J2-Pad3): track 30.3 -> 0.00 mm
- net Net-(J2-Pad4): track 27.9 -> 0.00 mm
- net SCL: track 25.8 -> 0.00 mm
- net SDA: track 25.5 -> 0.00 mm
- net Net-(R6-Pad2): track 25.3 -> 0.00 mm
- net Net-(R1-Pad2): track 16.0 -> 0.00 mm
- net Net-(R7-Pad1): track 7.58 -> 0.00 mm
- net Net-(R8-Pad2): track 5.13 -> 0.00 mm
Other:
- rule pad_to_mask_clearance: 0.051 -> 0
