File: attiny13-sensor/attiny13-sensor.sch (KiCad schematic (older format))
At the start: 5 parts, among them J1 Battery, J2 RX433_CONNECTOR, U1 ATtiny13A-PU, U2 DS18B20

Commit message: modified attiny project
Connections:
- net at R1.2, U2.2 (DQ): now also U1.6 (PB1); no longer U1.3 (PB4)
Changed lines of the file:
@@
 Connection ~ 5100 2250
-Wire Wire Line
-	5700 2950 6350 2950
-Wire Wire Line
-	6350 2950 6350 2850
-Connection ~ 6350 2850
 Wire Wire Line
 	6750 2250 7600 2250
@@
 $EndComp
 NoConn ~ 5700 2550
-NoConn ~ 5700 2650
 NoConn ~ 5700 2750
 NoConn ~ 5700 3050
@@
 	-1   0    0    1
 $EndComp
+Wire Wire Line
+	5700 2650 6350 2650
+Connection ~ 6350 2650
+NoConn ~ 5700 2950
 $EndSCHEMATC
