File: Lolin-nodemcu-v3-basestation/Lolin-nodemcu-v3-basestation.sch (KiCad schematic (older format))
At the start: 1 part

Commit message: нарисована базовая схема
Parts:
- added J1: RX433_CONNECTOR, symbol AlBalLib:RX433_CONNECTOR
- added J2: LCD1602_i2C_CONNECTOR, symbol AlBalLib:LCD1602_i2C_CONNECTOR
- added J3: BMP180_CONNECTOR, symbol AlBalLib:BMP180_CONNECTOR
- gave numbers to parts that had none: 1
Connections:
- net GND: now reaches U1.10 (GND)
- net GND: now also U1.14 (GND), U1.17 (GND), U1.2 (GND), U1.24 (GND), J1.4 (GND), J2.1 (GND), J3.2 (GND)
- net +5V: now reaches U1.15 (VIN_5V)
- net at U1.16 (3.3V): now also J3.1 (VIN)
- net at U1.22 (GPIO12): now also J2.3 (SDA), J3.4 (SDA)
- net at U1.23 (GPIO14): now also J2.4 (SCL), J3.3 (SCL)
- net at U1.27 (GPIO0): now also J1.3 (DATA)
- net VUSB: now reaches U1.3 (VUSB)
- net VUSB: now also J1.1 (VCC), J2.2 (VCC)
- no-connect marks 0 -> 20
